File: pcb/chakram-wheel/chakram-wheel.kicad_pcb (KiCad board)
At the start: 2 copper layers, 39.7 x 22.5 mm, 27 parts, among them J1 FPC Connector

Commit message: Added generated schematics, updated silkscreen and RGB board shape
Parts:
- removed the REF** at (87.5, 72.0)
- added REF**: Logo_Moucha_4.5x4.5mm_SilkScreen, Moucha_Graphics:Logo_Moucha_4.5x4.5mm_SilkScreen, B.Cu at (87.5, 71.5)
