File: pcb/chakram-wheel/chakram-wheel.kicad_sch (KiCad schematic)
At the start: 26 parts, among them J1 FPC Connector

Commit message: Added generated schematics, updated silkscreen and RGB board shape
Parts:
- EN1: footprint (none) -> Moucha_Primitives:RotaryEncoder_Alps_EC10E
Changed lines of the file:
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@@
 			)
 		)
-		(property "Footprint" ""
+		(property "Footprint" "Moucha_Primitives:RotaryEncoder_Alps_EC10E"
 			(at 157.226 39.37 0)
 			(effects
